Commit message: Update README with micromamba activation command and adjust joint origins in bracket_arm.urdf

File: urdf/bracket_arm.urdf (robot description, URDF)
Before this commit: robot bracket_arm, 7 links, 6 joints
Joints:
- joint joint_1: origin xyz=0 0 0.098 rpy=0 0 0 -> xyz=0 0 0.098 rpy=0 -1.5708 0
- joint joint_2: origin xyz=0 0 0.066 rpy=0 0 0 -> xyz=0 0 -0.066 rpy=0 0 0

Commit message: Fix joint_2 origin and axis parameters in bracket_arm.urdf for correct kinematics

File: urdf/bracket_arm.urdf (robot description, URDF)
Before this commit: robot bracket_arm, 7 links, 6 joints
Joints:
- joint joint_2: axis 0 1 0 -> 0 -1 0; origin xyz=0 0 -0.066 rpy=0 0 0 -> xyz=0 0 -0.066 rpy=0 -1.5708 0

Commit message: Add command and state interfaces with initial values for joints in bracket_arm.urdf

File: urdf/bracket_arm.urdf (robot description, URDF)
Before this commit: robot bracket_arm, 7 links, 6 joints
Joints:
- joint joint_3: origin xyz=0 0 0.103 rpy=0 3.1415 0 -> xyz=0 0 0.103 rpy=0 -1.5708 0

Commit message: Refactor joint parameters in bracket_arm.urdf and add initial_positions.yaml for joint configurations

File: urdf/bracket_arm.urdf (robot description, URDF)
Before this commit: robot bracket_arm, 7 links, 6 joints
Links:
- removed link gripper_tip_link
Joints:
- joint joint_2: origin xyz=0 0 -0.066 rpy=0 -1.5708 0 -> xyz=0 0 0.066 rpy=0 -1.5708 0

Commit message: Add gripper_tip_link and fix formatting in joint_5 definition in bracket_arm.urdf

File: urdf/bracket_arm.urdf (robot description, URDF)
Before this commit: robot bracket_arm, 6 links, 6 joints
Links:
- added link gripper_tip_link; visual box size=0.01 0.01 0.02

Commit message: Refactor bracket_arm.urdf: Update materials, adjust link dimensions, and correct joint definitions for improved accuracy

File: urdf/bracket_arm.urdf (robot description, URDF)
Before this commit: robot bracket_arm, 7 links, 6 joints
Links:
- removed link shoulder_link
- removed link wrist_pitch_link
- added link turret_link; visual cylinder length=0.082 radius=0.03
- added link wrist_link; visual cylinder length=0.103 radius=0.015
- link forearm_link: geometry visual cylinder length=0.066 radius=0.02
- link gripper_tip_link: geometry visual cylinder length=0.07 radius=0.01
- link upper_arm_link: geometry visual cylinder length=0.098 radius=0.02
Joints:
- joint joint_0: child shoulder_link -> turret_link; origin xyz=0 0 0.082 rpy=0 0 0 -> xyz=0 0 0.01 rpy=0 0 0
- joint joint_1: origin xyz=0 0 0.098 rpy=0 -1.5708 0 -> xyz=0 0 0.082 rpy=0 -1.5708 0; parent shoulder_link -> turret_link
- joint joint_2: origin xyz=0 0 0.066 rpy=0 -1.5708 0 -> xyz=0 0 0.098 rpy=0 0 0
- joint joint_3: child wrist_pitch_link -> wrist_link; origin xyz=0 0 0.103 rpy=0 -1.5708 0 -> xyz=0 0 0.066 rpy=0 0 0
- joint joint_4: origin xyz=0 0 0 rpy=0 0 0 -> xyz=0 0 0.103 rpy=0 0 0; parent wrist_pitch_link -> wrist_link
- joint joint_5: origin xyz=0 0 0.070 rpy=0 0.785 0 -> xyz=0 0 0.02 rpy=0 0.785 0

Commit message: Fix joint_2 parameters: update axis orientation and rotation for correct elbow movement

File: urdf/bracket_arm.urdf (robot description, URDF)
Before this commit: robot bracket_arm, 7 links, 6 joints
Joints:
- joint joint_2: axis 0 -1 0 -> 0 1 0; origin xyz=0 0 0.098 rpy=0 0 0 -> xyz=0 0 0.098 rpy=0 1.5708 0

Commit message: Fix joint_3 orientation: update rpy value for correct wrist movement and adjust initial position in configuration

File: urdf/bracket_arm.urdf (robot description, URDF)
Before this commit: robot bracket_arm, 7 links, 6 joints
Joints:
- joint joint_3: origin xyz=0 0 0.066 rpy=0 0 0 -> xyz=0 0 0.066 rpy=0 1.5708 0

Commit message: Fix joint_2 axis direction: invert axis for correct elbow rotation

File: urdf/bracket_arm.urdf (robot description, URDF)
Before this commit: robot bracket_arm, 7 links, 6 joints
Joints:
- joint joint_2: axis 0 1 0 -> 0 -1 0

Commit message: Fix joint_3 limit values: update range for correct wrist movement

File: urdf/bracket_arm.urdf (robot description, URDF)
Before this commit: robot bracket_arm, 7 links, 6 joints
Joints:
- joint joint_3: limit lower=-3.14 upper=0 effort=10 velocity=1.0 -> lower=0 upper=3.14 effort=10 velocity=1.0

Commit message: Fix joint limits and initial positions: update axis direction and adjust initial configuration for improved movement

File: urdf/bracket_arm.urdf (robot description, URDF)
Before this commit: robot bracket_arm, 7 links, 6 joints
Joints:
- joint joint_3: axis 0 1 0 -> 0 -1 0
- joint joint_4: limit lower=-1.57 upper=1.57 effort=10 velocity=1.0 -> lower=0 upper=3.14 effort=10 velocity=1.0
- joint joint_5: limit lower=0 upper=1.57 effort=10 velocity=1.0 -> lower=0 upper=3.14 effort=10 velocity=1.0

Commit message: Fix joint_3 parameters: update axis orientation and rotation for correct wrist movement

File: urdf/bracket_arm.urdf (robot description, URDF)
Before this commit: robot bracket_arm, 7 links, 6 joints
Joints:
- joint joint_3: axis 0 -1 0 -> 0 1 0; origin xyz=0 0 0.066 rpy=0 1.5708 0 -> xyz=0 0 0.066 rpy=0 -1.5708 0

Commit message: Fix joint_5 axis direction: invert axis for correct gripper rotation

File: urdf/bracket_arm.urdf (robot description, URDF)
Before this commit: robot bracket_arm, 7 links, 6 joints
Joints:
- joint joint_5: axis 0 1 0 -> 0 -1 0

Commit message: Fix joint_5 origin parameters: update rotation for correct gripper movement

File: urdf/bracket_arm.urdf (robot description, URDF)
Before this commit: robot bracket_arm, 7 links, 6 joints
Joints:
- joint joint_5: origin xyz=0 0 0.02 rpy=0 0.785 0 -> xyz=0 0 0.02 rpy=0 0 0

Commit message: Fix joint_5 origin and axis parameters: adjust position and invert axis for correct gripper movement

File: urdf/bracket_arm.urdf (robot description, URDF)
Before this commit: robot bracket_arm, 7 links, 6 joints
Links:
- added link gripper_finger_right_link; visual box size=0.01 0.005 0.04
Joints:
- added joint joint_5_mimic: type revolute, parent gripper_base_link, child gripper_finger_right_link, origin xyz=0 -0.015 0.02 rpy=0 0 0, axis 0 -1 0, limit lower=0 upper=3.14 effort=10 velocity=1.0, mimic joint=joint_5 multiplier=-1 offset=0
- joint joint_5: origin xyz=0 0 0.02 rpy=0 0 0 -> xyz=0 0.015 0.02 rpy=0 0 0

Commit message: Fix joint_5 origin parameters: adjust position for correct gripper alignment and update gripper finger dimensions

File: urdf/bracket_arm.urdf (robot description, URDF)
Before this commit: robot bracket_arm, 8 links, 7 joints
Links:
- link gripper_finger_right_link: geometry visual box size=0.02 0.01 0.07
Joints:
- joint joint_5: origin xyz=0 0.015 0.02 rpy=0 0 0 -> xyz=0 -0.015 0.02 rpy=0 0 0

Commit message: Fix joint_5 parameters: update child link and origin for correct finger positioning

File: urdf/bracket_arm.urdf (robot description, URDF)
Before this commit: robot bracket_arm, 8 links, 7 joints
Links:
- removed link gripper_tip_link
- added link gripper_finger_left_link; visual box size=0.02 0.01 0.07
Joints:
- joint joint_5: child gripper_tip_link -> gripper_finger_left_link; origin xyz=0 -0.015 0.02 rpy=0 0 0 -> xyz=-0.02 0.015 0.0 rpy=0 0 0
- joint joint_5_mimic: origin xyz=0 -0.015 0.02 rpy=0 0 0 -> xyz=0.02 0.015 0.0 rpy=0 0 0

Commit message: Fix joint_5 parameters: update limits and origin for improved finger positioning

File: urdf/bracket_arm.urdf (robot description, URDF)
Before this commit: robot bracket_arm, 8 links, 7 joints
Joints:
- joint joint_0: limit lower=-1.57 upper=1.57 effort=10 velocity=1.0 -> lower=0 upper=3.14 effort=10 velocity=1.0
- joint joint_5: origin xyz=-0.02 0.015 0.0 rpy=0 0 0 -> xyz=-0.01 0.01 0.0 rpy=0 0 0
- joint joint_5_mimic: origin xyz=0.02 0.015 0.0 rpy=0 0 0 -> xyz=0.01 0.01 0.0 rpy=0 0 0

Commit message: Fix upper arm link geometry: replace cylinder with box for improved representation

File: urdf/bracket_arm.urdf (robot description, URDF)
Before this commit: robot bracket_arm, 8 links, 7 joints
Links:
- link upper_arm_link: geometry visual box size=0.04 0.02 0.098

Commit message: Fix geometry representation: replace cylinder with box for upper arm, forearm, and wrist links

File: urdf/bracket_arm.urdf (robot description, URDF)
Before this commit: robot bracket_arm, 8 links, 7 joints
Links:
- link forearm_link: geometry visual box size=0.02 0.04 0.066
- link upper_arm_link: geometry visual box size=0.02 0.04 0.098
- link wrist_link: geometry visual box size=0.04 0.02 0.103

Commit message: Fix visual representation: update box size for base link, adjust cylinder radius and material for turret link, and change material for upper arm link

File: urdf/bracket_arm.urdf (robot description, URDF)
Before this commit: robot bracket_arm, 8 links, 7 joints
Links:
- link base_link: geometry collision box size=0.15 0.15 0.005; visual box size=0.5 0.5 0.005
- link forearm_link: geometry collision box size=0.02 0.04 0.066; visual box size=0.02 0.04 0.066
- link gripper_base_link: geometry collision box size=0.03 0.03 0.02; visual box size=0.03 0.03 0.02
- link gripper_finger_left_link: geometry collision box size=0.02 0.01 0.07; visual box size=0.02 0.01 0.07
- link gripper_finger_right_link: geometry collision box size=0.02 0.01 0.07; visual box size=0.02 0.01 0.07
- link turret_link: geometry collision cylinder length=0.082 radius=0.056; visual cylinder length=0.082 radius=0.056
- link upper_arm_link: geometry collision box size=0.02 0.04 0.098; visual box size=0.02 0.04 0.098
- link wrist_link: geometry collision box size=0.04 0.02 0.103; visual box size=0.04 0.02 0.103

Commit message: Update initial joint positions and add TCP joint for wrist link in URDF

File: urdf/bracket_arm.urdf (robot description, URDF)
Before this commit: robot bracket_arm, 8 links, 7 joints
Links:
- added link tcp_link
Joints:
- added joint joint_tcp: type fixed, parent wrist_link, child tcp_link, origin xyz=0 0 0.103 rpy=0 0 0

Commit message: Refactor action server implementation and update TCP joint configuration in URDF

File: urdf/bracket_arm.urdf (robot description, URDF)
Before this commit: robot bracket_arm, 9 links, 8 joints
Joints:
- joint joint_tcp: origin xyz=0 0 0.103 rpy=0 0 0 -> xyz=0 0 0 rpy=0 0 0; parent wrist_link -> gripper_base_link

Commit message: Update joint limits in bracket_arm.urdf for increased precision

File: urdf/bracket_arm.urdf (robot description, URDF)
Before this commit: robot bracket_arm, 9 links, 8 joints
Joints:
- joint joint_0: limit lower=0 upper=3.14 effort=10 velocity=1.0 -> lower=0 upper=3.14160 effort=10 velocity=1.0
- joint joint_1: limit lower=0 upper=3.14 effort=10 velocity=1.0 -> lower=0 upper=3.14160 effort=10 velocity=1.0
- joint joint_2: limit lower=0 upper=3.14 effort=10 velocity=1.0 -> lower=0 upper=3.14160 effort=10 velocity=1.0
- joint joint_3: limit lower=0 upper=3.14 effort=10 velocity=1.0 -> lower=0 upper=3.14160 effort=10 velocity=1.0
- joint joint_4: limit lower=0 upper=3.14 effort=10 velocity=1.0 -> lower=0 upper=3.14160 effort=10 velocity=1.0
- joint joint_5: limit lower=0 upper=3.14 effort=10 velocity=1.0 -> lower=0 upper=3.14160 effort=10 velocity=1.0
- joint joint_5_mimic: limit lower=0 upper=3.14 effort=10 velocity=1.0 -> lower=0 upper=3.14160 effort=10 velocity=1.0

Commit message: Add grasp joint and link for improved IK/Perception reference

File: urdf/bracket_arm.urdf (robot description, URDF)
Before this commit: robot bracket_arm, 9 links, 8 joints
Links:
- added link grasp_link
Joints:
- added joint joint_grasp: type fixed, parent gripper_base_link, child grasp_link, origin xyz=0 0.01 0.05 rpy=0 0 0

Commit message: Add grasp joint and link for improved IK/Perception reference

File: urdf/bracket_arm.urdf (robot description, URDF)
Before this commit: robot bracket_arm, 10 links, 9 joints
Joints:
- joint joint_grasp: origin xyz=0 0.01 0.05 rpy=0 0 0 -> xyz=0 0.01 0.07 rpy=0 0 0

Commit message: Add service setup and deployment scripts for BA Arm ROS2 Bridge

File: urdf/bracket_arm.urdf (robot description, URDF)
Before this commit: robot bracket_arm, 10 links, 9 joints
Links:
- added link marker_base
- added link marker_forearm
- added link marker_grasp
Joints:
- added joint joint_marker_base: type fixed, parent base_link, child marker_base, origin xyz=0.05 0.0 0.005 rpy=0 0 0
- added joint joint_marker_forearm: type fixed, parent forearm_link, child marker_forearm, origin xyz=0 0 0.033 rpy=0 0 0
- added joint joint_marker_grasp: type fixed, parent gripper_base_link, child marker_grasp, origin xyz=0 0 0.02 rpy=0 0 0

Commit message: Adjust marker joint origins for improved alignment in URDF model

File: urdf/bracket_arm.urdf (robot description, URDF)
Before this commit: robot bracket_arm, 13 links, 12 joints
Joints:
- joint joint_marker_base: origin xyz=0.05 0.0 0.005 rpy=0 0 0 -> xyz=0.095 0.065 0.005 rpy=0 0 0
- joint joint_marker_forearm: origin xyz=0 0 0.033 rpy=0 0 0 -> xyz=0 0.01 0.11 rpy=0 0 0
- joint joint_marker_grasp: origin xyz=0 0 0.02 rpy=0 0 0 -> xyz=0 0.025 0.02 rpy=0 0 0

Commit message: Adjust marker joint origins for improved alignment in URDF model

File: urdf/bracket_arm.urdf (robot description, URDF)
Before this commit: robot bracket_arm, 13 links, 12 joints
Joints:
- joint joint_marker_base: origin xyz=0.095 0.065 0.005 rpy=0 0 0 -> xyz=0.095 0.065 0.015 rpy=0 0 0
- joint joint_marker_forearm: origin xyz=0 0.01 0.11 rpy=0 0 0 -> xyz=0 0.02 0.11 rpy=0 0 0
- joint joint_marker_grasp: origin xyz=0 0.025 0.02 rpy=0 0 0 -> xyz=0 0.03 0.02 rpy=0 0 0

Commit message: urdf fix.

File: urdf/bracket_arm.urdf (robot description, URDF)
Before this commit: robot bracket_arm, 13 links, 12 joints
Links:
- link gripper_base_link: geometry collision box size=0.03 0.03 0.03; visual box size=0.03 0.03 0.03
- link marker_base: geometry visual sphere radius=0.009
- link marker_forearm: geometry visual sphere radius=0.009
- link marker_grasp: geometry visual sphere radius=0.009
- link upper_arm_link: geometry collision box size=0.02 0.04 0.10; visual box size=0.02 0.04 0.10
- link wrist_link: geometry collision box size=0.04 0.02 0.072; visual box size=0.04 0.02 0.072
Joints:
- joint joint_2: origin xyz=0 0 0.098 rpy=0 1.5708 0 -> xyz=0 0 0.10 rpy=0 1.5708 0
- joint joint_4: origin xyz=0 0 0.103 rpy=0 0 0 -> xyz=0 0 0.072 rpy=0 0 0
- joint joint_5: origin xyz=-0.01 0.01 0.0 rpy=0 0 0 -> xyz=-0.01 0.01 0.03 rpy=0 0 0
- joint joint_5_mimic: origin xyz=0.01 0.01 0.0 rpy=0 0 0 -> xyz=0.01 0.01 0.03 rpy=0 0 0
- joint joint_grasp: origin xyz=0 0.01 0.07 rpy=0 0 0 -> xyz=0 0.01 0.10 rpy=0 0 0
- joint joint_marker_base: origin xyz=0.095 0.065 0.015 rpy=0 0 0 -> xyz=-0.095 0.065 0.015 rpy=0 0 0
- joint joint_marker_forearm: origin xyz=0 0.02 0.11 rpy=0 0 0 -> xyz=-0.02 0 0.05 rpy=0 0 0; parent forearm_link -> wrist_link
- joint joint_marker_grasp: origin xyz=0 0.03 0.02 rpy=0 0 0 -> xyz=0 0.03 0.05 rpy=0 0 0

Commit message: add joint_overview_camera

File: urdf/bracket_arm.urdf (robot description, URDF)
Before this commit: robot bracket_arm, 13 links, 12 joints
Links:
- added link overview_camera_link
Joints:
- added joint joint_overview_camera: type fixed, parent base_link, child overview_camera_link, origin xyz=-0.16 0.17 0.34 rpy=-2.678 0 -1.5708

Commit message: urdf update.

File: urdf/bracket_arm.urdf (robot description, URDF)
Before this commit: robot bracket_arm, 14 links, 13 joints
Links:
- removed link overview_camera_link
- added link overview_camera_nominal
- link forearm_link: geometry collision box size=0.02 0.04 0.065; visual box size=0.02 0.04 0.065
- link upper_arm_link: geometry collision box size=0.02 0.04 0.098; visual box size=0.02 0.04 0.098
- link wrist_link: geometry collision box size=0.04 0.02 0.070; visual box size=0.04 0.02 0.070
Joints:
- removed joint joint_overview_camera
- added joint joint_overview_camera_nominal: type fixed, parent base_link, child overview_camera_nominal, origin xyz=-0.16 0.17 0.34 rpy=-2.678 0 -1.5708
- joint joint_1: origin xyz=0 0 0.082 rpy=0 -1.5708 0 -> xyz=-0.008 0 0.082 rpy=0 -1.5708 0
- joint joint_2: origin xyz=0 0 0.10 rpy=0 1.5708 0 -> xyz=0 0 0.098 rpy=0 1.5708 0
- joint joint_3: origin xyz=0 0 0.066 rpy=0 -1.5708 0 -> xyz=0 0 0.065 rpy=0 -1.5708 0
- joint joint_4: origin xyz=0 0 0.072 rpy=0 0 0 -> xyz=0 0 0.070 rpy=0 0 0
- joint joint_marker_base: origin xyz=-0.095 0.065 0.015 rpy=0 0 0 -> xyz=-0.098 0.065 0.016 rpy=0 0 0
- joint joint_marker_forearm: origin xyz=-0.02 0 0.05 rpy=0 0 0 -> xyz=-0.022 0 0.049 rpy=0 0 0
- joint joint_marker_grasp: origin xyz=0 0.03 0.05 rpy=0 0 0 -> xyz=0 0.034 0.05 rpy=0 0 0

Commit message: Fix IndexError in debug log for single-point trajectories

File: urdf/bracket_arm.urdf (robot description, URDF)
Before this commit: robot bracket_arm, 14 links, 13 joints
Joints:
- joint joint_5_mimic: limit lower=0 upper=3.14160 effort=10 velocity=1.0 -> lower=-3.1416 upper=0 effort=10 velocity=1.0
